File: OpenHAK_Display.kicad_pcb (KiCad board)
At the start: 2 copper layers, 23.4 x 21.7 mm, 13 parts, among them P1 M52-Series_Male_TH_Harwin

Commit message: updated layout of BETA Display branch
Parts:
- P1: footprint Solutions:M52-Series_M_TH_0.05_Harwin -> Solutions:M52-Series_M_TH_0.05_8POS_Harwin
- moved P1 2.54 mm to (136.4, 111.9)
- turned C5 to 270 degrees
- turned C6 to 90 degrees
Connections:
- C5 pad 1: +3V3 -> GND
- C5 pad 2: GND -> +3V3
- C6 pad 1: +3V3 -> GND
- C6 pad 2: GND -> +3V3
- P1 pad 1: GND -> Net-(P1-Pad1)
- P1 pad 2: +3V3 -> /SDA
- P1 pad 4: /SDA -> /SCL
- P1 pad 6: /SCL -> /OLED_RST
- P1 pad 7: Net-(P1-Pad7) -> +3V3
- P1 pad 8: /OLED_RST -> GND
Routing:
- net GND: track 2.18 -> 1.50 mm, vias 0 -> 1
