File: OpenHAK_Display.sch (KiCad schematic (older format))
At the start: 11 parts, among them P1 M52-Series_Male_TH_Harwin

Commit message: changed tx rx on schematics
Other:
- note added: "OpenHAK Display Master Branch"
- note added: "PIN 21\nPIN 24\nPIN 25\nSIM_RX\nPIN2\nSIM_TX\nPIN 3\nRST\nVDD\nGND"
- note removed: "PIN 21\nPIN 24\nPIN 25\nUART TX\nPIN2\nUART RX\nPIN 3\nRST\nVDD\nGND"
Changed lines of the file:
@@
 EESchema Schematic File Version 4
+LIBS:OpenHAK_Display-cache
 EELAYER 26 0
 EELAYER END
@@
 $EndComp
 Text Notes 7750 4300 0    70   ~ 0
-PIN 21\nPIN 24\nPIN 25\nUART TX\nPIN2\nUART RX\nPIN 3\nRST\nVDD\nGND
+PIN 21\nPIN 24\nPIN 25\nSIM_RX\nPIN2\nSIM_TX\nPIN 3\nRST\nVDD\nGND
 $Comp
 L power:GND #PWR04
@@
 Text Label 3550 4250 0    50   ~ 0
 VCC
+Text Notes 5050 2350 0    50   ~ 0
+OpenHAK Display Master Branch
 $EndSCHEMATC
