File: OpenHAK_Display.sch (KiCad schematic (older format))
At the start: 10 parts, among them P1 CONN_01X08

Commit message: swapped 0603 for 0402
Parts:
- C1, C2, C3, C4, C5, C6, R1, R2: footprint Capacitors_SMD:C_0603 -> Capacitors_SMD:C_0402
Changed lines of the file:
@@
 F 0 "C1" H 3160 3470 50  0000 L CNN
 F 1 "1uF" H 3160 3320 50  0000 L CNN
-F 2 "Capacitors_SMD:C_0603" H 3150 3400 50  0001 C CNN
+F 2 "Capacitors_SMD:C_0402" H 3150 3400 50  0001 C CNN
 F 3 "" H 3150 3400 50  0000 C CNN
 	1    3150 3400
@@
 F 0 "C2" H 3160 3820 50  0000 L CNN
 F 1 "1uF" H 3160 3670 50  0000 L CNN
-F 2 "Capacitors_SMD:C_0603" H 3150 3750 50  0001 C CNN
+F 2 "Capacitors_SMD:C_0402" H 3150 3750 50  0001 C CNN
 F 3 "" H 3150 3750 50  0000 C CNN
 	1    3150 3750
@@
 F 0 "R2" H 3430 2620 50  0000 L CNN
 F 1 "10K" H 3430 2560 50  0000 L CNN
-F 2 "Capacitors_SMD:C_0603" H 3400 2600 50  0001 C CNN
+F 2 "Capacitors_SMD:C_0402" H 3400 2600 50  0001 C CNN
 F 3 "" H 3400 2600 50  0000 C CNN
 	1    3400 2600
@@
 F 0 "C4" H 3560 4870 50  0000 L CNN
 F 1 "2.2uF" H 3560 4720 50  0000 L CNN
-F 2 "Capacitors_SMD:C_0603" H 3550 4800 50  0001 C CNN
+F 2 "Capacitors_SMD:C_0402" H 3550 4800 50  0001 C CNN
 F 3 "" H 3550 4800 50  0000 C CNN
 	1    3550 4800
@@
 F 0 "C3" H 3260 4870 50  0000 L CNN
 F 1 "4.7uF 16V" H 3100 4700 50  0000 L CNN
-F 2 "Capacitors_SMD:C_0603" H 3250 4800 50  0001 C CNN
+F 2 "Capacitors_SMD:C_0402" H 3250 4800 50  0001 C CNN
 F 3 "" H 3250 4800 50  0000 C CNN
 	1    3250 4800
@@
 F 0 "R1" H 2980 4820 50  0000 L CNN
 F 1 "390K" H 2980 4760 50  0000 L CNN
-F 2 "Capacitors_SMD:C_0603" H 2950 4800 50  0001 C CNN
+F 2 "Capacitors_SMD:C_0402" H 2950 4800 50  0001 C CNN
 F 3 "" H 2950 4800 50  0000 C CNN
 	1    2950 4800
@@
 F 0 "C5" V 7200 3050 50  0000 L CNN
 F 1 "1uF" V 7200 2800 50  0000 L CNN
-F 2 "Capacitors_SMD:C_0603" H 7150 3000 50  0001 C CNN
+F 2 "Capacitors_SMD:C_0402" H 7150 3000 50  0001 C CNN
 F 3 "" H 7150 3000 50  0000 C CNN
 	1    7150 3000
@@
 F 0 "C6" V 7200 3200 50  0000 L CNN
 F 1 "0.1uF" V 7250 2950 50  0000 L CNN
-F 2 "Capacitors_SMD:C_0603" H 7150 3150 50  0001 C CNN
+F 2 "Capacitors_SMD:C_0402" H 7150 3150 50  0001 C CNN
 F 3 "" H 7150 3150 50  0000 C CNN
 	1    7150 3150

Commit message: updating layout to fit beta board
Parts:
- LCD1: symbol Solutions1:OLED_64x48 -> OpenHAK_Display:OpenHAK_Display_Solutions1_OLED_64x48
- P1: value CONN_01X08 -> M52-Series_Male_TH_Harwin; footprint Solutions:8_pin_Castellation_127 -> Solutions:M52-Series_M_TH_0.05_Harwin; symbol OpenHAK_Display-rescue:CONN_01X08 -> Connector:Conn_01x10_Male
Connections:
- wire segments 62 -> 58
- no-connect marks 11 -> 13
Other:
- note added: "PIN 21\nPIN 24\nPIN 25\nUART TX\nPIN2\nUART RX\nPIN 3\nRST\nVDD\nGND"
- note removed: "GND\n3V3\nPIN 25\nUART TX\nPIN2\nUART RX\nPIN 3\nRST"
- moved on the sheet: C5, C6
Changed lines of the file:
@@
 $EndDescr
 $Comp
-L Solutions1:OLED_64x48 LCD1
+L OpenHAK_Display:OpenHAK_Display_Solutions1_OLED_64x48 LCD1
 U 1 1 5A64ECF1
 P 4350 3700
@@
 L power:+3V3 #PWR02
 U 1 1 5A64EEC3
-P 6900 2900
-F 0 "#PWR02" H 6900 2750 50  0001 C CNN
-F 1 "+3V3" H 6900 3040 50  0000 C CNN
-F 2 "" H 6900 2900 50  0000 C CNN
-F 3 "" H 6900 2900 50  0000 C CNN
-	1    6900 2900
+P 7000 4100
+F 0 "#PWR02" H 7000 3950 50  0001 C CNN
+F 1 "+3V3" H 7000 4240 50  0000 C CNN
+F 2 "" H 7000 4100 50  0000 C CNN
+F 3 "" H 7000 4100 50  0000 C CNN
+	1    7000 4100
 	1    0    0    -1
 $EndComp
@@
 SDA
 $Comp
-L OpenHAK_Display-rescue:CONN_01X08 P1
+L Connector:Conn_01x10_Male P1
 U 1 1 5A64F98A
-P 7650 3650
-F 0 "P1" H 7650 4100 50  0000 C CNN
-F 1 "CONN_01X08" V 7750 3650 50  0000 C CNN
-F 2 "Solutions:8_pin_Castellation_127" H 7650 3650 50  0001 C CNN
-F 3 "" H 7650 3650 50  0000 C CNN
-	1    7650 3650
-	1    0    0    -1
-$EndComp
-Text Notes 7850 4050 0    70   ~ 0
-GND\n3V3\nPIN 25\nUART TX\nPIN2\nUART RX\nPIN 3\nRST
+P 7650 3800
+F 0 "P1" H 7650 4250 50  0000 C CNN
+F 1 "M52-Series_Male_TH_Harwin" H 7900 3150 50  0000 C CNN
+F 2 "Solutions:M52-Series_M_TH_0.05_Harwin" H 7650 3800 50  0001 C CNN
+F 3 "" H 7650 3800 50  0000 C CNN
+	1    7650 3800
+	-1   0    0    1
+$EndComp
+Text Notes 7750 4300 0    70   ~ 0
+PIN 21\nPIN 24\nPIN 25\nUART TX\nPIN2\nUART RX\nPIN 3\nRST\nVDD\nGND
 $Comp
 L power:GND #PWR04
 U 1 1 5A64FAC1
-P 7500 2950
-F 0 "#PWR04" H 7500 2700 50  0001 C CNN
-F 1 "GND" H 7500 2800 50  0000 C CNN
-F 2 "" H 7500 2950 50  0000 C CNN
-F 3 "" H 7500 2950 50  0000 C CNN
-	1    7500 2950
-	1    0    0    -1
-$EndComp
-Wire Wire Line
-	7350 3300 7450 3300
-Wire Wire Line
-	7350 2900 7350 3000
-Wire Wire Line
-	7350 2900 7500 2900
-Wire Wire Line
-	7500 2900 7500 2950
-Wire Wire Line
-	7450 3400 6900 3400
-Wire Wire Line
-	6900 3400 6900 3150
+P 7400 4400
+F 0 "#PWR04" H 7400 4150 50  0001 C CNN
+F 1 "GND" H 7400 4250 50  0000 C CNN
+F 2 "" H 7400 4400 50  0000 C CNN
+F 3 "" H 7400 4400 50  0000 C CNN
+	1    7400 4400
+	1    0    0    -1
+$EndComp
 NoConn ~ 7450 3600
 NoConn ~ 7450 3800
@@
 L Device:C_Small C5
 U 1 1 5A6762A1
-P 7150 3000
-F 0 "C5" V 7200 3050 50  0000 L CNN
-F 1 "1uF" V 7200 2800 50  0000 L CNN
-F 2 "Capacitors_SMD:C_0402" H 7150 3000 50  0001 C CNN
-F 3 "" H 7150 3000 50  0000 C CNN
-	1    7150 3000
-	0    1    -1   0
+P 7000 4250
+F 0 "C5" H 7050 4350 50  0000 L CNN
+F 1 "1uF" H 7050 4150 50  0000 L CNN
+F 2 "Capacitors_SMD:C_0402" H 7000 4250 50  0001 C CNN
+F 3 "" H 7000 4250 50  0000 C CNN
+	1    7000 4250
+	-1   0    0    -1
 $EndComp
 $Comp
 L Device:C_Small C6
 U 1 1 5A676327
-P 7150 3150
-F 0 "C6" V 7200 3200 50  0000 L CNN
-F 1 "0.1uF" V 7250 2950 50  0000 L CNN
-F 2 "Capacitors_SMD:C_0402" H 7150 3150 50  0001 C CNN
-F 3 "" H 7150 3150 50  0000 C CNN
-	1    7150 3150
-	0    1    1    0
-$EndComp
-Wire Wire Line
-	7050 3000 6900 3000
-Connection ~ 6900 3000
-Wire Wire Line
-	7050 3150 6900 3150
-Connection ~ 6900 3150
-Wire Wire Line
-	7250 3000 7350 3000
-Connection ~ 7350 3000
-Wire Wire Line
-	7250 3150 7350 3150
-Connection ~ 7350 3150
+P 7200 4250
+F 0 "C6" H 7100 4350 50  0000 L CNN
+F 1 "0.1uF" H 7000 4150 50  0000 L CNN
+F 2 "Capacitors_SMD:C_0402" H 7200 4250 50  0001 C CNN
+F 3 "" H 7200 4250 50  0000 C CNN
+	1    7200 4250
+	1    0    0    -1
+$EndComp
 Wire Wire Line
 	5050 3800 5150 3800
@@
 	3550 5150 3650 5150
 Wire Wire Line
-	6900 3000 6900 2900
-Wire Wire Line
-	6900 3150 6900 3000
-Wire Wire Line
-	7350 3000 7350 3150
-Wire Wire Line
-	7350 3150 7350 3300
-Wire Wire Line
 	5150 3700 5300 3700
+Wire Wire Line
+	7450 4100 7200 4100
+Wire Wire Line
+	7000 4100 7000 4150
+Wire Wire Line
+	7200 4150 7200 4100
+Connection ~ 7200 4100
+Wire Wire Line
+	7200 4100 7000 4100
+Wire Wire Line
+	7000 4350 7000 4400
+Wire Wire Line
+	7000 4400 7200 4400
+Wire Wire Line
+	7400 4400 7400 4200
+Wire Wire Line
+	7400 4200 7450 4200
+Wire Wire Line
+	7200 4350 7200 4400
+Connection ~ 7200 4400
+Wire Wire Line
+	7200 4400 7400 4400
+Connection ~ 7400 4400
+Connection ~ 7000 4100
+NoConn ~ 7450 3300
+NoConn ~ 7450 3400
 $EndSCHEMATC

Commit message: cleaned up silk and made production files
Parts:
- added C7: TEST POINT, Capacitors_SMD:C_0805, symbol Device:C_Small
Connections:
- net labels added: VCC
- wire segments 58 -> 60
Changed lines of the file:
@@
 EESchema Schematic File Version 4
-LIBS:OpenHAK_Display-cache
 EELAYER 26 0
 EELAYER END
@@
 NoConn ~ 7450 3300
 NoConn ~ 7450 3400
+$Comp
+L Device:C_Small C7
+U 1 1 5D07F71A
+P 5850 4450
+F 0 "C7" H 5900 4350 50  0000 L CNN
+F 1 "TEST POINT" H 5900 4550 50  0000 L CNN
+F 2 "Capacitors_SMD:C_0805" H 5850 4450 50  0001 C CNN
+F 3 "" H 5850 4450 50  0000 C CNN
+	1    5850 4450
+	-1   0    0    -1
+$EndComp
+Text Label 5850 4250 0    50   ~ 0
+VCC
+Wire Wire Line
+	5850 4350 5850 4250
+Wire Wire Line
+	5850 4550 5850 4650
+$Comp
+L power:GND #PWR05
+U 1 1 5D08272A
+P 5850 4650
+F 0 "#PWR05" H 5850 4400 50  0001 C CNN
+F 1 "GND" H 5850 4500 50  0000 C CNN
+F 2 "" H 5850 4650 50  0000 C CNN
+F 3 "" H 5850 4650 50  0000 C CNN
+	1    5850 4650
+	1    0    0    -1
+$EndComp
+Text Label 3550 4250 0    50   ~ 0
+VCC
 $EndSCHEMATC

Commit message: made production files
Parts:
- C3: footprint Capacitors_SMD:C_0402 -> Capacitors_SMD:C_0603
Changed lines of the file:
@@
 F 0 "C3" H 3260 4870 50  0000 L CNN
 F 1 "4.7uF 16V" H 3100 4700 50  0000 L CNN
-F 2 "Capacitors_SMD:C_0402" H 3250 4800 50  0001 C CNN
+F 2 "Capacitors_SMD:C_0603" H 3250 4800 50  0001 C CNN
 F 3 "" H 3250 4800 50  0000 C CNN
 	1    3250 4800

Commit message: updating beta branch
Parts:
- P1: symbol Connector:Conn_01x10_Male -> Connector:Conn_01x08_Male
Connections:
- wire segments 60 -> 63
- no-connect marks 13 -> 11
Other:
- note added: "GND\nVDD\nPIN 25\nSIM_RX\nPIN2\nSIM_TX\nPIN 3\nRST\n"
- note added: "OpenHAK Display\nBETA BRANCH"
- note removed: "PIN 21\nPIN 24\nPIN 25\nUART TX\nPIN2\nUART RX\nPIN 3\nRST\nVDD\nGND"
- moved on the sheet: C5, C6
Changed lines of the file:
@@
 EESchema Schematic File Version 4
+LIBS:OpenHAK_Display-cache
 EELAYER 26 0
 EELAYER END
@@
 L power:+3V3 #PWR02
 U 1 1 5A64EEC3
-P 7000 4100
-F 0 "#PWR02" H 7000 3950 50  0001 C CNN
-F 1 "+3V3" H 7000 4240 50  0000 C CNN
-F 2 "" H 7000 4100 50  0000 C CNN
-F 3 "" H 7000 4100 50  0000 C CNN
-	1    7000 4100
+P 6900 3250
+F 0 "#PWR02" H 6900 3100 50  0001 C CNN
+F 1 "+3V3" H 6900 3390 50  0000 C CNN
+F 2 "" H 6900 3250 50  0000 C CNN
+F 3 "" H 6900 3250 50  0000 C CNN
+	1    6900 3250
 	1    0    0    -1
 $EndComp
@@
 SDA
 $Comp
-L Connector:Conn_01x10_Male P1
+L Connector:Conn_01x08_Male P1
 U 1 1 5A64F98A
-P 7650 3800
-F 0 "P1" H 7650 4250 50  0000 C CNN
-F 1 "M52-Series_Male_TH_Harwin" H 7900 3150 50  0000 C CNN
-F 2 "Solutions:M52-Series_M_TH_0.05_Harwin" H 7650 3800 50  0001 C CNN
-F 3 "" H 7650 3800 50  0000 C CNN
-	1    7650 3800
+P 7650 3700
+F 0 "P1" H 7650 4150 50  0000 C CNN
+F 1 "M52-Series_Male_TH_Harwin" H 7500 3100 50  0000 C CNN
+F 2 "Solutions:M52-Series_M_TH_0.05_Harwin" H 7650 3700 50  0001 C CNN
+F 3 "" H 7650 3700 50  0000 C CNN
+	1    7650 3700
 	-1   0    0    1
 $EndComp
-Text Notes 7750 4300 0    70   ~ 0
-PIN 21\nPIN 24\nPIN 25\nUART TX\nPIN2\nUART RX\nPIN 3\nRST\nVDD\nGND
+Text Notes 7700 4050 0    70   ~ 0
+GND\nVDD\nPIN 25\nSIM_RX\nPIN2\nSIM_TX\nPIN 3\nRST\n
 $Comp
 L power:GND #PWR04
 U 1 1 5A64FAC1
-P 7400 4400
-F 0 "#PWR04" H 7400 4150 50  0001 C CNN
-F 1 "GND" H 7400 4250 50  0000 C CNN
-F 2 "" H 7400 4400 50  0000 C CNN
-F 3 "" H 7400 4400 50  0000 C CNN
-	1    7400 4400
+P 6250 3650
+F 0 "#PWR04" H 6250 3400 50  0001 C CNN
+F 1 "GND" H 6250 3500 50  0000 C CNN
+F 2 "" H 6250 3650 50  0000 C CNN
+F 3 "" H 6250 3650 50  0000 C CNN
+	1    6250 3650
 	1    0    0    -1
 $EndComp
@@
 L Device:C_Small C5
 U 1 1 5A6762A1
-P 7000 4250
-F 0 "C5" H 7050 4350 50  0000 L CNN
-F 1 "1uF" H 7050 4150 50  0000 L CNN
-F 2 "Capacitors_SMD:C_0402" H 7000 4250 50  0001 C CNN
-F 3 "" H 7000 4250 50  0000 C CNN
-	1    7000 4250
+P 6500 3450
+F 0 "C5" H 6550 3550 50  0000 L CNN
+F 1 "1uF" H 6550 3350 50  0000 L CNN
+F 2 "Capacitors_SMD:C_0402" H 6500 3450 50  0001 C CNN
+F 3 "" H 6500 3450 50  0000 C CNN
+	1    6500 3450
 	-1   0    0    -1
 $EndComp
@@
 L Device:C_Small C6
 U 1 1 5A676327
-P 7200 4250
-F 0 "C6" H 7100 4350 50  0000 L CNN
-F 1 "0.1uF" H 7000 4150 50  0000 L CNN
-F 2 "Capacitors_SMD:C_0402" H 7200 4250 50  0001 C CNN
-F 3 "" H 7200 4250 50  0000 C CNN
-	1    7200 4250
+P 6700 3450
+F 0 "C6" H 6600 3550 50  0000 L CNN
+F 1 "0.1uF" H 6500 3350 50  0000 L CNN
+F 2 "Capacitors_SMD:C_0402" H 6700 3450 50  0001 C CNN
+F 3 "" H 6700 3450 50  0000 C CNN
+	1    6700 3450
 	1    0    0    -1
 $EndComp
@@
 	5150 3700 5300 3700
 Wire Wire Line
-	7450 4100 7200 4100
-Wire Wire Line
-	7000 4100 7000 4150
-Wire Wire Line
-	7200 4150 7200 4100
-Connection ~ 7200 4100
-Wire Wire Line
-	7200 4100 7000 4100
-Wire Wire Line
-	7000 4350 7000 4400
-Wire Wire Line
-	7000 4400 7200 4400
-Wire Wire Line
-	7400 4400 7400 4200
-Wire Wire Line
-	7400 4200 7450 4200
-Wire Wire Line
-	7200 4350 7200 4400
-Connection ~ 7200 4400
-Wire Wire Line
-	7200 4400 7400 4400
-Connection ~ 7400 4400
-Connection ~ 7000 4100
-NoConn ~ 7450 3300
-NoConn ~ 7450 3400
+	7450 3300 6700 3300
+Wire Wire Line
+	6500 3300 6500 3350
+Wire Wire Line
+	6700 3350 6700 3300
+Connection ~ 6700 3300
+Wire Wire Line
+	6700 3300 6500 3300
+Wire Wire Line
+	6500 3550 6500 3600
+Wire Wire Line
+	6500 3600 6700 3600
+Wire Wire Line
+	6900 3600 6900 3400
+Wire Wire Line
+	6900 3400 7450 3400
+Wire Wire Line
+	6700 3550 6700 3600
+Connection ~ 6700 3600
+Wire Wire Line
+	6700 3600 6900 3600
+Connection ~ 6500 3300
 $Comp
 L Device:C_Small C7
@@
 Text Label 3550 4250 0    50   ~ 0
 VCC
+Text Notes 5750 2550 0    50   ~ 0
+OpenHAK Display\nBETA BRANCH
+Wire Wire Line
+	6250 3650 6250 3300
+Wire Wire Line
+	6250 3300 6500 3300
+Wire Wire Line
+	6900 3250 6900 3400
+Connection ~ 6900 3400
 $EndSCHEMATC

Commit message: updated layout of BETA Display branch
Parts:
- P1: footprint Solutions:M52-Series_M_TH_0.05_Harwin -> Solutions:M52-Series_M_TH_0.05_8POS_Harwin
Changed lines of the file:
@@
 F 0 "P1" H 7650 4150 50  0000 C CNN
 F 1 "M52-Series_Male_TH_Harwin" H 7500 3100 50  0000 C CNN
-F 2 "Solutions:M52-Series_M_TH_0.05_Harwin" H 7650 3700 50  0001 C CNN
+F 2 "Solutions:M52-Series_M_TH_0.05_8POS_Harwin" H 7650 3700 50  0001 C CNN
 F 3 "" H 7650 3700 50  0000 C CNN
 	1    7650 3700
